Commit message: Agrega simulación y control para NuestroRobot4

File: src/NuestroRobot4/urdf/NuestroRobot4.urdf (robot description, URDF)
Before this commit: robot NuestroRobot4, 7 links, 6 joints
Links:
- added link world
Joints:
- added joint base_joint: type fixed, parent world, child base_link, origin xyz=0.0 0.0 0.0 rpy=0 0 0
- joint Joint_Right: mimic (none) -> joint=Joint_Left multiplier=-1 offset=0
